Commit message: Add camera to description

File: turtlebot_unizar_description/robots/kobuki_hexagons_hokuyo_top.urdf.xacro (robot description, xacro)
@@ -9,4 +9,7 @@
   <xacro:stack_hexagons                 parent="base_link"/>
   <xacro:sensor_hokuyo          	      parent="plate_top_link"/>
-  <xacro:sensor_d435i                   parent="plate_top_link"/>
+  <xacro:gimbal                         parent="plate_top_link"/>
+  <xacro:sensor_d435i                   parent="camera_mount_gimbal_link">
+    <origin xyz="0 0 0" rpy="0 0 0"/>
+  </xacro:sensor_d435i>
 </robot>

File: turtlebot_unizar_description/urdf/sensors/gimbal.urdf.xacro (robot description, xacro)
@@ -1,12 +1,12 @@
 <?xml version="1.0"?>
-<robot name="sensor_hokuyo" xmlns:xacro="http://ros.org/wiki/xacro">
+<robot name="gimbal_struct" xmlns:xacro="http://ros.org/wiki/xacro">
 	<xacro:include filename="$(find turtlebot_description)/urdf/turtlebot_gazebo.urdf.xacro"/>
 	<xacro:include filename="$(find turtlebot_description)/urdf/turtlebot_properties.urdf.xacro"/>
-	<xacro:macro name="sensor_hokuyo" params="parent">
-		<link name="base_laser_plate_link">
+	<xacro:macro name="gimbal" params="parent">
+		<link name="base_gimbal_plate_link">
 			<collision>
 				<origin xyz="0 0 0" rpy="0 0 0"/>
 				<geometry>
-					<box size="0.084 0.084 0.004" />
+					<box size="0.18 0.18 0.011" />
 				</geometry>
 			</collision>
@@ -14,5 +14,5 @@
 				<origin xyz="0 0 0" rpy="0 0 0"/>
 				<geometry>
-				<box size="0.084 0.084 0.004" />
+					<box size="0.18 0.18 0.011" />
 				</geometry>
 				<material name="Gray">
@@ -26,11 +26,11 @@
 			</inertial>
 		</link>
-		<joint name="hokuyo_plate_joint" type="fixed">
+		<joint name="gimbal_plate_joint" type="fixed">
 			<axis xyz="0 0 1" />
-			<origin xyz="0.227 0.0 0.005" rpy="0 0 0"/>
+			<origin xyz="0.095 0.0 0.0055" rpy="0 0 0"/>
 			<parent link="${parent}"/>
-			<child link="base_laser_plate_link"/>
+			<child link="base_gimbal_plate_link"/>
 		</joint>
-		<link name="base_laser_link">
+		<link name="base_gimbal_link">
 			<collision>
 				<origin xyz="0 0 0" rpy="0 0 0"/>
@@ -42,6 +42,9 @@
 				<origin xyz="0 0 0" rpy="0 0 0"/>
 				<geometry>
-					<mesh filename="package://turtlebot_description/meshes/sensors/hokuyo.dae"/>
+					<box size="0.034 0.034 0.1935" />
 				</geometry>
+				<material name="Gray">
+					<color rgba="0.5 0.5 0.5 1"/>
+				</material>
 			</visual>
 			<inertial>
@@ -51,9 +54,17 @@
 			</inertial>
 		</link>
-		<joint name="hokuyo_joint" type="fixed">
+		<joint name="gimbal_joint" type="fixed">
 			<axis xyz="0 0 1" />
-			<origin xyz="0 0.0 0.037" rpy="0 0 0"/>
-			<parent link="base_laser_plate_link"/>
-			<child link="base_laser_link"/>
+			<origin xyz="0 0.0 0.09675" rpy="0 0 0"/>
+			<parent link="base_gimbal_plate_link"/>
+			<child link="base_gimbal_link"/>
+		</joint>
+		<link name="camera_mount_gimbal_link">
+		</link>
+		<joint name="camera_mount_gimbal_joint" type="fixed">
+			<axis xyz="0 0 1" />
+			<origin xyz="0 0.0 0.09675" rpy="0 0 0"/>
+			<parent link="base_gimbal_link"/>
+			<child link="camera_mount_gimbal_link"/>
 		</joint>
 	</xacro:macro>

File: turtlebot_unizar_description/urdf/turtlebot_library.urdf.xacro (robot description, xacro)
@@ -14,4 +14,6 @@
   <!-- Hokuyo Laser -->
   <xacro:include filename="$(find turtlebot_unizar_description)/urdf/sensors/hokuyo.urdf.xacro"/>
+  <!-- Gimbal -->
+  <xacro:include filename="$(find turtlebot_unizar_description)/urdf/sensors/gimbal.urdf.xacro"/>
   <!-- Realsense -->
   <xacro:include filename="$(find realsense2_description)/urdf/_d435i.urdf.xacro"/>
